Commit message: feat: roarm_m3.urdf를 업데이트하고 프리미티브 형상 추가
불완전한 roarm_m3.urdf 파일을 roarm_m3_complete.urdf의 내용으로 업데이트했습니다.

STL 메시 파일을 찾거나 생성할 수 없어 프리미티브 형상을 사용하도록 시각적 및 충돌 형상을 수정했습니다. URDF 파일은 이제 완전하며 시뮬레이션에 사용할 수 있습니다.

File: assets/roarm_m3/urdf/roarm_m3.urdf (robot description, URDF)
Before this commit: robot roarm_m3, 7 links, 6 joints
Links:
- removed link link_base
- removed link link_elbow
- removed link link_gripper
- removed link link_shoulder
- removed link link_wrist1
- removed link link_wrist2
- added link gripper_link, mass 0.0028708; collision box size=0.02 0.02 0.06; visual box size=0.02 0.02 0.06
- added link hand_tcp, mass 0.0005; collision sphere radius=0.01; visual sphere radius=0.01
- added link link1, mass 0.0729177; collision cylinder length=0.05 radius=0.03; visual cylinder length=0.05 radius=0.03
- added link link2, mass 0.0703216; collision cylinder length=0.15 radius=0.02; visual cylinder length=0.15 radius=0.02
- added link link3, mass 0.021608; collision cylinder length=0.15 radius=0.02; visual cylinder length=0.15 radius=0.02
- added link link4, mass 0.0099933; collision cylinder length=0.12 radius=0.018; visual cylinder length=0.12 radius=0.018
- added link link5, mass 0.0153928; collision cylinder length=0.08 radius=0.015; visual cylinder length=0.08 radius=0.015
- added link world
- link base_link: mass 1.0 -> 0.2562183
Joints:
- removed joint joint_base
- removed joint joint_elbow
- removed joint joint_gripper
- removed joint joint_shoulder
- removed joint joint_wrist1
- removed joint joint_wrist2
- added joint base_link_to_link1: type revolute, parent base_link, child link1, origin xyz=0.0 0.0 0.0 rpy=0 0 0, axis 0 0 1, limit lower=-3.1416 upper=3.1416 effort=10.0 velocity=2.0
- added joint link1_to_link2: type revolute, parent link1, child link2, origin xyz=0.0 0.0 0.051959 rpy=-1.5708 -1.5708 0, axis 0 0 1, limit lower=-1.5708 upper=1.5708 effort=15.0 velocity=2.0
- added joint link2_to_link3: type revolute, parent link2, child link3, origin xyz=0.236815 0.030002 0 rpy=0 0 1.5708, axis 0 0 1, limit lower=-1.0 upper=2.95 effort=10.0 velocity=2.5
- added joint link3_to_link4: type revolute, parent link3, child link4, origin xyz=0.0 -0.144586 0 rpy=0 0 0, axis 0 0 1, limit lower=-1.5708 upper=1.5708 effort=8.0 velocity=3.0
- added joint link4_to_link5: type revolute, parent link4, child link5, origin xyz=0.015147 -0.053653 0 rpy=1.5708 1.5708 0, axis 0 0 1, limit lower=-3.1416 upper=3.1416 effort=5.0 velocity=3.5
- added joint link5_to_gripper_link: type revolute, parent link5, child gripper_link, origin xyz=0.0 0.018821 0.052035 rpy=-1.5708 -1.5708 0, axis 0 0 1, limit lower=0.0 upper=1.5 effort=5.0 velocity=3.0
- added joint link5_to_hand_tcp: type fixed, parent link5, child hand_tcp, origin xyz=0 0 0.115428 rpy=1.5708 -1.5708 0, axis 0 0 0
- added joint world_to_base_link: type fixed, parent world, child base_link, origin xyz=0.0 0.0 0.0701 rpy=0 0 0, axis 0 0 1
