Commit message: feat(v3.7.3): Joint limit expansion experiment and gripper fix
Changes:
- URDF: Expanded joint limits from ±90° to ±180° (v3.7.3 experiment)
- Environment: Fixed gripper width observation bug (obs[23] now uses tracked_width)
- Training: Added comprehensive logging and monitoring

Results (100K steps):
- REACH: 11.0% (down from 36.2% in v3.7.2)
- Min distance: 28.0cm (vs 5.5cm in v3.7.2)
- Value loss: 0.0123 (stable)

Root Cause Analysis:
- 4x exploration space expansion (±90°→±180°) requires >400K training steps
- 100K steps insufficient for new space exploration
- Gripper width bug successfully fixed and verified

Testing:
- Added test_v3_7_2.py for direct environment testing
- Created tests/test_gripper.py with comprehensive unit tests
- Validated gripper width tracking and state management

Documentation:
- logs/v3.7.3_FINAL_SUMMARY.md: Quick reference summary
- logs/v3.7.3_progress_summary.md: Detailed experiment analysis
- README.md: Updated with v3.7.3 results and v3.7.4 plan

Configuration:
- Updated .gitignore to exclude checkpoints and tensorboard files

Next Steps (v3.7.4):
- Revert URDF to ±90° joint limits
- Keep gripper width fix
- Expected: REACH 36%+, potential GRIP achievement

File: assets/roarm_m3/urdf/roarm_m3_multiprim.urdf (robot description, URDF)
Before this commit: robot roarm_m3_multiprim, 10 links, 9 joints
Links:
- link gripper_left_finger: mass 0.0080 -> 0.0100; geometry collision box size=0.020 0.010 0.010; collision cylinder length=0.030 radius=0.006
- link gripper_right_finger: mass 0.0080 -> 0.0100; geometry collision box size=0.020 0.010 0.010; collision cylinder length=0.030 radius=0.006
Joints:
- joint gripper_left_joint: limit lower=0 upper=0.02 effort=5 velocity=0.05 -> lower=0 upper=0.025 effort=8 velocity=0.08
- joint gripper_right_joint: limit lower=0 upper=0.02 effort=5 velocity=0.05 -> lower=0 upper=0.025 effort=8 velocity=0.08
- joint joint_2: limit lower=-1.57 upper=1.57 effort=15 velocity=1.5 -> lower=-3.14159 upper=3.14159 effort=15 velocity=1.5
- joint joint_3: limit lower=-1.57 upper=1.57 effort=10 velocity=2.0 -> lower=-3.14159 upper=3.14159 effort=10 velocity=2.0
- joint joint_4: limit lower=-1.57 upper=1.57 effort=8 velocity=2.5 -> lower=-3.14159 upper=3.14159 effort=8 velocity=2.5
- joint joint_6: limit lower=-1.57 upper=1.57 effort=3 velocity=2.0 -> lower=-3.14159 upper=3.14159 effort=3 velocity=2.0

Commit message: v3.9.0: Robust GRIP 시스템 구현 (False Positive 방지)
ChatGPT 피드백 반영:
- 성공 정의: Attach & Lift & Hold (물리적 부착 확인)
- 보상/평가 분리: 느슨한 보상 vs 엄격한 성공 조건
- 단계별 지표: reach_rate, attach_rate, lift_rate, success_rate

코드 변경:
- envs/roarm_pick_place_env.py
  * ENV_VERSION v3.9.0 선언
  * 메트릭 구조 재설계 (first_attach, first_lift, success)
  * initial_cube_z 저장 (리프트 계산용)
  * is_attached 기반 성공 정의 구현
  * Milestone Rewards 재설계 (REACH/ATTACH/LIFT/SUCCESS)

새 파일:
- scripts/rl/validate_grip_quality.py (False Positive 검증 도구)
- docs/v3.9.0_robust_grip_plan.md (전략 문서)
- docs/v3.9.0_implementation_report.md (구현 보고서)

목표:
- False Positive < 10%
- Attach 성공률 20-40%
- v3.8.1 대비 안정적인 GRIP 평가

File: assets/roarm_m3/urdf/roarm_m3_multiprim.urdf (robot description, URDF)
Before this commit: robot roarm_m3_multiprim, 10 links, 9 joints
Joints:
- joint joint_2: limit lower=-3.14159 upper=3.14159 effort=15 velocity=1.5 -> lower=-1.57 upper=1.57 effort=15 velocity=1.5
- joint joint_3: limit lower=-3.14159 upper=3.14159 effort=10 velocity=2.0 -> lower=-1.57 upper=1.57 effort=10 velocity=2.0
- joint joint_6: limit lower=-3.14159 upper=3.14159 effort=3 velocity=2.0 -> lower=-1.57 upper=1.57 effort=3 velocity=2.0
